File: person-keyboard.kicad_pcb (KiCad board)
At the start: 2 copper layers, 233 parts, among them SW1 esc, SW10 f9, SW100 R ctrl, SW101 Left, SW102 down, SW103 right, SW104 num zero, SW105 num full stop, SW11 f10, SW12 f11, SW13 f12, SW14 prtscr, SW15 scrlck, SW16 pause, SW17 tilde, SW18 1, SW19 2, SW2 f1, SW20 3, SW21 4, SW22 5, SW23 6, SW24 7, SW25 8, SW26 9, SW27 0, SW28 minus, SW29 equals, SW3 f2, SW30 backspace, SW31 insert, SW32 home, SW33 pgup, SW34 num lock, SW35 num slash, SW36 num mult, SW37 num minus, SW38 tab, SW39 q, SW4 f3, SW40 w, SW41 e, SW42 r, SW43 t, SW44 y, SW45 u, SW46 i, SW47 o, SW48 p, SW49 L brac, SW5 f4, SW50 R brac, SW51 enter, SW52 delete, SW53 end, SW54 pgdn, SW55 num 7, SW56 num 8, SW57 num 9, SW58 num add, SW59 capslock, SW6 f5, SW60 a, SW61 s, SW62 d, SW63 f, SW64 g, SW65 h, SW66 j, SW67 k, SW68 l, SW69 sem colon, SW7 f6, SW70 quote, SW71 tilde, SW72 num 4, SW73 num 5, SW74 num 6, SW75 L shift, SW76 backslash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

Commit message: Starting work
Parts:
- moved D10 30.0 mm to (269.4, 67.1)
- moved D28 30.0 mm to (269.4, 95.7)
- moved SW21 30.0 mm to (130.9, 91.7)
- moved D18 30.0 mm to (78.9, 95.7)
- moved D59 30.0 mm to (67.0, 133.8)
- moved SW18 30.0 mm to (73.8, 91.7)
- moved SW86 30.0 mm to (269.0, 148.8)
- moved D100 30.0 mm to (324.1, 171.9)
- moved D101 30.0 mm to (350.3, 171.9)
- moved D102 30.0 mm to (369.4, 171.9)
- moved D103 30.0 mm to (388.4, 171.9)
- moved D104 30.0 mm to (421.8, 171.9)
- moved D105 30.0 mm to (450.3, 171.9)
- moved D17 30.0 mm to (59.8, 95.7)
- moved D19 30.0 mm to (97.9, 95.7)
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Other:
- board outline added: 446.9 x 141.7 mm

Commit message: Fixed key matrix, laid out LED matrix, started laying out microcontroller
Parts:
- added C1: 10u, Capacitor_SMD:C_0805_2012Metric, F.Cu at (451.2, 41.7)
- added C2: 22u, Capacitor_SMD:C_0805_2012Metric, F.Cu at (451.2, 44.7)
- added F1: 500mA, Fuse:Fuse_0805_2012Metric, F.Cu at (446.8, 37.3)
- added J1: USB_C_Receptacle_USB2.0_16P, Connector_USB:USB_C_Receptacle_GCT_USB4105-xx-A_16P_TopMnt_Horizontal, B.Cu at (408.4, 23.4)
- added R1: 5k2, Resistor_SMD:R_0805_2012Metric, F.Cu at (446.8, 40.3)
- added R2: 5k1, Resistor_SMD:R_0805_2012Metric, F.Cu at (446.8, 43.2)
- added R6: 1M, Resistor_SMD:R_0805_2012Metric, F.Cu at (446.8, 46.2)
- added R8: 1k, Resistor_SMD:R_0402_1005Metric, B.Cu at (393.2, 46.0)
- added SK1: SK6812MINI, Keebio-Parts:SK6812-MINI-E, B.Cu at (38.1, 43.1)
- added SK10: SK6812MINI, Keebio-Parts:SK6812-MINI-E, B.Cu at (247.7, 43.1)
- added SK100: SK6812MINI, Keebio-Parts:SK6812-MINI-E, B.Cu at (302.4, 147.9)
- added SK101: SK6812MINI, Keebio-Parts:SK6812-MINI-E, B.Cu at (328.6, 147.9)
- added SK102: SK6812MINI, Keebio-Parts:SK6812-MINI-E, B.Cu at (347.7, 147.9)
- added SK103: SK6812MINI, Keebio-Parts:SK6812-MINI-E, B.Cu at (366.7, 147.9)
- added SK104: SK6812MINI, Keebio-Parts:SK6812-MINI-E, B.Cu at (400.1, 147.9)
- added SK105: SK6812MINI, Keebio-Parts:SK6812-MINI-E, B.Cu at (428.6, 147.9)
- added SK11: SK6812MINI, Keebio-Parts:SK6812-MINI-E, B.Cu at (266.7, 43.1)
- added SK12: SK6812MINI, Keebio-Parts:SK6812-MINI-E, B.Cu at (285.8, 43.1)
- added SK13: SK6812MINI, Keebio-Parts:SK6812-MINI-E, B.Cu at (304.8, 43.1)
- added SK14: SK6812MINI, Keebio-Parts:SK6812-MINI-E, B.Cu at (328.6, 43.1)
- added SK15: SK6812MINI, Keebio-Parts:SK6812-MINI-E, B.Cu at (347.7, 43.1)
- added SK16: SK6812MINI, Keebio-Parts:SK6812-MINI-E, B.Cu at (366.7, 43.1)
- added SK17: SK6812MINI, Keebio-Parts:SK6812-MINI-E, B.Cu at (38.1, 71.7)
- added SK18: SK6812MINI, Keebio-Parts:SK6812-MINI-E, B.Cu at (57.1, 71.7)
- added SK19: SK6812MINI, Keebio-Parts:SK6812-MINI-E, B.Cu at (76.2, 71.7)
- added SK2: SK6812MINI, Keebio-Parts:SK6812-MINI-E, B.Cu at (76.2, 43.1)
- added SK20: SK6812MINI, Keebio-Parts:SK6812-MINI-E, B.Cu at (95.2, 71.7)
- added SK21: SK6812MINI, Keebio-Parts:SK6812-MINI-E, B.Cu at (114.3, 71.7)
- added SK22: SK6812MINI, Keebio-Parts:SK6812-MINI-E, B.Cu at (133.3, 71.7)
- added SK23: SK6812MINI, Keebio-Parts:SK6812-MINI-E, B.Cu at (152.4, 71.7)
- added SK24: SK6812MINI, Keebio-Parts:SK6812-MINI-E, B.Cu at (171.4, 71.7)
- added SK25: SK6812MINI, Keebio-Parts:SK6812-MINI-E, B.Cu at (190.5, 71.7)
- added SK26: SK6812MINI, Keebio-Parts:SK6812-MINI-E, B.Cu at (209.6, 71.7)
- added SK27: SK6812MINI, Keebio-Parts:SK6812-MINI-E, B.Cu at (228.6, 71.7)
- added SK28: SK6812MINI, Keebio-Parts:SK6812-MINI-E, B.Cu at (247.7, 71.7)
- added SK29: SK6812MINI, Keebio-Parts:SK6812-MINI-E, B.Cu at (266.7, 71.7)
- added SK3: SK6812MINI, Keebio-Parts:SK6812-MINI-E, B.Cu at (95.2, 43.1)
- added SK30: SK6812MINI, Keebio-Parts:SK6812-MINI-E, B.Cu at (295.3, 71.7)
- added SK31: SK6812MINI, Keebio-Parts:SK6812-MINI-E, B.Cu at (328.6, 71.7)
- added SK32: SK6812MINI, Keebio-Parts:SK6812-MINI-E, B.Cu at (347.7, 71.7)
- added SK33: SK6812MINI, Keebio-Parts:SK6812-MINI-E, B.Cu at (366.7, 71.7)
- added SK34: SK6812MINI, Keebio-Parts:SK6812-MINI-E, B.Cu at (390.5, 71.7)
- added SK35: SK6812MINI, Keebio-Parts:SK6812-MINI-E, B.Cu at (409.6, 71.7)
- added SK36: SK6812MINI, Keebio-Parts:SK6812-MINI-E, B.Cu at (428.6, 71.7)
- added SK37: SK6812MINI, Keebio-Parts:SK6812-MINI-E, B.Cu at (447.7, 71.7)
- added SK38: SK6812MINI, Keebio-Parts:SK6812-MINI-E, B.Cu at (42.9, 90.7)
- added SK39: SK6812MINI, Keebio-Parts:SK6812-MINI-E, B.Cu at (66.7, 90.7)
- added SK4: SK6812MINI, Keebio-Parts:SK6812-MINI-E, B.Cu at (114.3, 43.1)
- added SK40: SK6812MINI, Keebio-Parts:SK6812-MINI-E, B.Cu at (85.7, 90.7)
- added SK41: SK6812MINI, Keebio-Parts:SK6812-MINI-E, B.Cu at (104.8, 90.7)
- added SK42: SK6812MINI, Keebio-Parts:SK6812-MINI-E, B.Cu at (123.8, 90.7)
- added SK43: SK6812MINI, Keebio-Parts:SK6812-MINI-E, B.Cu at (142.9, 90.7)
- added SK44: SK6812MINI, Keebio-Parts:SK6812-MINI-E, B.Cu at (161.9, 90.7)
- added SK45: SK6812MINI, Keebio-Parts:SK6812-MINI-E, B.Cu at (181.0, 90.7)
- added SK46: SK6812MINI, Keebio-Parts:SK6812-MINI-E, B.Cu at (200.0, 90.7)
- added SK47: SK6812MINI, Keebio-Parts:SK6812-MINI-E, B.Cu at (219.1, 90.7)
- added SK48: SK6812MINI, Keebio-Parts:SK6812-MINI-E, B.Cu at (238.1, 90.7)
- added SK49: SK6812MINI, Keebio-Parts:SK6812-MINI-E, B.Cu at (257.2, 90.7)
- added SK5: SK6812MINI, Keebio-Parts:SK6812-MINI-E, B.Cu at (133.3, 43.1)
- added SK50: SK6812MINI, Keebio-Parts:SK6812-MINI-E, B.Cu at (276.2, 90.7)
- added SK51: SK6812MINI, Keebio-Parts:SK6812-MINI-E, B.Cu at (302.4, 100.2)
- added SK52: SK6812MINI, Keebio-Parts:SK6812-MINI-E, B.Cu at (328.6, 90.7)
- added SK53: SK6812MINI, Keebio-Parts:SK6812-MINI-E, B.Cu at (347.7, 90.7)
- added SK54: SK6812MINI, Keebio-Parts:SK6812-MINI-E, B.Cu at (366.7, 90.7)
- added SK55: SK6812MINI, Keebio-Parts:SK6812-MINI-E, B.Cu at (390.5, 90.7)
- added SK56: SK6812MINI, Keebio-Parts:SK6812-MINI-E, B.Cu at (409.6, 90.7)
- added SK57: SK6812MINI, Keebio-Parts:SK6812-MINI-E, B.Cu at (428.6, 90.7)
- added SK58: SK6812MINI, Keebio-Parts:SK6812-MINI-E, B.Cu at (447.7, 100.2)
- added SK59: SK6812MINI, Keebio-Parts:SK6812-MINI-E, B.Cu at (45.2, 109.8)
- added SK6: SK6812MINI, Keebio-Parts:SK6812-MINI-E, B.Cu at (161.9, 43.1)
- added SK60: SK6812MINI, Keebio-Parts:SK6812-MINI-E, B.Cu at (71.4, 109.8)
- added SK61: SK6812MINI, Keebio-Parts:SK6812-MINI-E, B.Cu at (90.5, 109.8)
- added SK62: SK6812MINI, Keebio-Parts:SK6812-MINI-E, B.Cu at (109.5, 109.8)
- added SK63: SK6812MINI, Keebio-Parts:SK6812-MINI-E, B.Cu at (128.6, 109.8)
- added SK64: SK6812MINI, Keebio-Parts:SK6812-MINI-E, B.Cu at (147.6, 109.8)
- added SK65: SK6812MINI, Keebio-Parts:SK6812-MINI-E, B.Cu at (166.7, 109.8)
- added SK66: SK6812MINI, Keebio-Parts:SK6812-MINI-E, B.Cu at (185.7, 109.8)
- added SK67: SK6812MINI, Keebio-Parts:SK6812-MINI-E, B.Cu at (204.8, 109.8)
- added SK68: SK6812MINI, Keebio-Parts:SK6812-MINI-E, B.Cu at (223.8, 109.8)
- added SK69: SK6812MINI, Keebio-Parts:SK6812-MINI-E, B.Cu at (242.9, 109.8)
- added SK7: SK6812MINI, Keebio-Parts:SK6812-MINI-E, B.Cu at (181.0, 43.1)
- added SK70: SK6812MINI, Keebio-Parts:SK6812-MINI-E, B.Cu at (261.9, 109.8)
- added SK71: SK6812MINI, Keebio-Parts:SK6812-MINI-E, B.Cu at (281.0, 109.8)
- added SK72: SK6812MINI, Keebio-Parts:SK6812-MINI-E, B.Cu at (390.5, 109.8)
- added SK73: SK6812MINI, Keebio-Parts:SK6812-MINI-E, B.Cu at (409.6, 109.8)
- added SK74: SK6812MINI, Keebio-Parts:SK6812-MINI-E, B.Cu at (428.6, 109.8)
- added SK75: SK6812MINI, Keebio-Parts:SK6812-MINI-E, B.Cu at (40.5, 128.8)
- added SK76: SK6812MINI, Keebio-Parts:SK6812-MINI-E, B.Cu at (61.9, 128.8)
- added SK77: SK6812MINI, Keebio-Parts:SK6812-MINI-E, B.Cu at (81.0, 128.8)
- added SK78: SK6812MINI, Keebio-Parts:SK6812-MINI-E, B.Cu at (100.0, 128.8)
- added SK79: SK6812MINI, Keebio-Parts:SK6812-MINI-E, B.Cu at (119.1, 128.8)
- added SK8: SK6812MINI, Keebio-Parts:SK6812-MINI-E, B.Cu at (200.0, 43.1)
- added SK80: SK6812MINI, Keebio-Parts:SK6812-MINI-E, B.Cu at (138.1, 128.8)
- added SK81: SK6812MINI, Keebio-Parts:SK6812-MINI-E, B.Cu at (157.2, 128.8)
- added SK82: SK6812MINI, Keebio-Parts:SK6812-MINI-E, B.Cu at (176.2, 128.8)
- added SK83: SK6812MINI, Keebio-Parts:SK6812-MINI-E, B.Cu at (195.3, 128.8)
- added SK84: SK6812MINI, Keebio-Parts:SK6812-MINI-E, B.Cu at (214.3, 128.8)
- added SK85: SK6812MINI, Keebio-Parts:SK6812-MINI-E, B.Cu at (233.4, 128.8)
- added SK86: SK6812MINI, Keebio-Parts:SK6812-MINI-E, B.Cu at (252.4, 128.8)
- added SK87: SK6812MINI, Keebio-Parts:SK6812-MINI-E, B.Cu at (288.1, 128.8)
- added SK88: SK6812MINI, Keebio-Parts:SK6812-MINI-E, B.Cu at (347.7, 128.8)
- added SK89: SK6812MINI, Keebio-Parts:SK6812-MINI-E, B.Cu at (390.5, 128.8)
- added SK9: SK6812MINI, Keebio-Parts:SK6812-MINI-E, B.Cu at (219.1, 43.1)
- added SK90: SK6812MINI, Keebio-Parts:SK6812-MINI-E, B.Cu at (409.6, 128.8)
- added SK91: SK6812MINI, Keebio-Parts:SK6812-MINI-E, B.Cu at (428.6, 128.8)
- added SK92: SK6812MINI, Keebio-Parts:SK6812-MINI-E, B.Cu at (447.7, 138.3)
- added SK93: SK6812MINI, Keebio-Parts:SK6812-MINI-E, B.Cu at (40.5, 147.9)
- added SK94: SK6812MINI, Keebio-Parts:SK6812-MINI-E, B.Cu at (64.3, 147.9)
- added SK95: SK6812MINI, Keebio-Parts:SK6812-MINI-E, B.Cu at (88.1, 147.9)
- added SK96: SK6812MINI, Keebio-Parts:SK6812-MINI-E, B.Cu at (159.5, 147.9)
- added SK97: SK6812MINI, Keebio-Parts:SK6812-MINI-E, B.Cu at (231.0, 147.9)
- added SK98: SK6812MINI, Keebio-Parts:SK6812-MINI-E, B.Cu at (254.8, 147.9)
- added SK99: SK6812MINI, Keebio-Parts:SK6812-MINI-E, B.Cu at (278.6, 147.9)
- added SW107: SW_Push, jacob-libs:SW-SMD_L4.0-W2.9-LS5.0, F.Cu at (452.3, 38.0)
- added U5: 74AHCT1G125, Package_TO_SOT_SMD:SOT-23-5_HandSoldering, F.Cu at (54.8, 43.7)
- C10, C11, C12, C13, C14, C15, C16, C17, C4, C5, C6, C7, C8, C9, D1, D10, D100, D101, D102, D103, D104, D105, D11, D12, D13, D14, D15, D16, D17, D18, D19, D2, D20, D21, D22, D23, D24, D25, D26, D27, D28, D29, D3, D30, D31, D32, D33, D34, D35, D36, D37, D38, D39, D4, D40, D41, D42, D43, D44, D45, D46, D47, D48, D49, D5, D50, D51, D52, D53, D54, D55, D56, D57, D58, D59, D6, D60, D61, D62, D63, D64, D65, D66, D67, D68, D69, D7, D70, D71, D72, D73, D74, D75, D76, D77, D78, D79, D8, D80, D81, D82, D83, D84, D85, D86, D87, D88, D89, D9, D90, D91, D92, D93, D94, D95, D96, D97, D98, D99, R3, R4, R5, R7, U1, U2, U3, U4, Y1: moved to B.Cu
- moved R7 175.3 mm to (438.7, 46.0), turned to 180 degrees
- moved U2 173.2 mm to (430.4, 39.9), turned to 180 degrees
- moved C14 173.2 mm to (424.1, 36.7), turned to 180 degrees
- moved C17 173.2 mm to (424.1, 42.6), turned to 180 degrees
- moved C10 173.2 mm to (421.2, 38.6), turned to 180 degrees
- moved C11 173.2 mm to (421.2, 40.6), turned to 180 degrees
- moved C12 173.2 mm to (421.2, 42.6), turned to 180 degrees
- moved C13 173.2 mm to (421.2, 44.5), turned to 180 degrees
- moved C4 173.2 mm to (418.3, 36.7), turned to 180 degrees
- moved C5 173.2 mm to (418.3, 38.6), turned to 180 degrees
- moved C6 173.2 mm to (418.3, 40.6), turned to 180 degrees
- moved C7 173.2 mm to (418.3, 42.6), turned to 180 degrees
- moved C8 173.2 mm to (418.3, 44.5), turned to 180 degrees
- moved C9 173.2 mm to (421.2, 36.7), turned to 180 degrees
- moved R3 173.2 mm to (419.3, 47.0), turned to 180 degrees
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Connections:
- C15 pad 2: Net-(U1-XOUT) -> Net-(C15-Pad2)
- D87 pad 1: row8 -> row9
- R3 pad 1: unconnected-(R3-Pad1) -> Net-(R3-Pad1)
- SW105 pad 1: Net-(SW105-Pad1) -> col9
- SW36 pad 1: Net-(SW105-Pad1) -> col9
- SW37 pad 1: Net-(SW105-Pad1) -> col9
- SW57 pad 1: Net-(SW105-Pad1) -> col9
- SW58 pad 1: Net-(SW105-Pad1) -> col9
- SW74 pad 1: Net-(SW105-Pad1) -> col9
- SW87 pad 1: col7 -> col6
- SW91 pad 1: Net-(SW105-Pad1) -> col9
- SW92 pad 1: Net-(SW105-Pad1) -> col9
- Y1 pad 4: Net-(U1-XOUT) -> Net-(C15-Pad2)
Routing:
- net /d+: track 0.00 -> 13.5 mm
- net /d-: track 0.00 -> 12.6 mm
- net Net-(D71-A): track 0.00 -> 7.38 mm
- net Net-(D53-A): track 0.00 -> 7.38 mm
- net Net-(D52-A): track 0.00 -> 7.38 mm
- net Net-(D50-A): track 0.00 -> 7.38 mm
- net Net-(D49-A): track 0.00 -> 7.38 mm
- net Net-(D37-A): track 0.00 -> 7.38 mm
- net Net-(D32-A): track 0.00 -> 7.38 mm
- net Net-(D31-A): track 0.00 -> 7.38 mm
- net Net-(D104-A): track 0.00 -> 7.38 mm
- net Net-(D102-A): track 0.00 -> 7.38 mm
- net Net-(D101-A): track 0.00 -> 7.38 mm
- net Net-(D15-A): track 0.00 -> 7.38 mm
- net Net-(D14-A): track 0.00 -> 7.38 mm
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Other:
- outline, holes or cut-outs redrawn

Commit message: Added protection diode, reconsidered mcu position
Parts:
- added D106: B340A, PCM_Diode_SMD_AKL:D_SMA, B.Cu at (396.0, 22.9)
- added R9: 1R, Resistor_SMD:R_0805_2012Metric_Pad1.20x1.40mm_HandSolder, B.Cu at (402.5, 29.3)
- C1, C2: footprint Capacitor_SMD:C_0805_2012Metric -> Capacitor_SMD:C_0805_2012Metric_Pad1.18x1.45mm_HandSolder; moved to B.Cu
- C10, C11, C12, C13, C14, C15, C16, C17, C4, C5, C6, C7, C8, C9: footprint Capacitor_SMD:C_0402_1005Metric -> Capacitor_SMD:C_0402_1005Metric_Pad0.74x0.62mm_HandSolder
- F1, R6, U5: moved to B.Cu
- R1: value 5k2 -> 5k1; footprint Resistor_SMD:R_0805_2012Metric -> Resistor_SMD:R_0805_2012Metric_Pad1.20x1.40mm_HandSolder; moved to B.Cu
- R2: footprint Resistor_SMD:R_0805_2012Metric -> Resistor_SMD:R_0805_2012Metric_Pad1.20x1.40mm_HandSolder; moved to B.Cu
- R8: footprint Resistor_SMD:R_0402_1005Metric -> Resistor_SMD:R_0402_1005Metric_Pad0.72x0.64mm_HandSolder
- moved C2 50.6 mm to (402.4, 31.4)
- moved U2 36.1 mm to (395.9, 29.3), turned to 0 degrees
- moved SW107 27.3 mm to (425.4, 42.7)
- moved U3 26.7 mm to (411.2, 47.2), turned to -90 degrees
- moved C10 18.6 mm to (433.7, 24.9)
- moved C11 18.6 mm to (433.7, 26.9)
- moved C12 18.6 mm to (433.7, 28.9)
- moved C13 18.6 mm to (433.7, 30.8)
- moved C14 18.6 mm to (436.6, 22.9)
- moved C17 18.6 mm to (436.6, 28.9)
- moved C4 18.6 mm to (430.9, 22.9)
- moved C5 18.6 mm to (430.9, 24.9)
- moved C6 18.6 mm to (430.9, 26.9)
- moved C7 18.6 mm to (430.9, 28.9)
- moved C8 18.6 mm to (430.9, 30.8)
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Connections:
- C2 pad 1: +3V3 -> Net-(C2-Pad1)
- F1 pad 2: +5V -> Net-(D106-A)
Routing:
- net /d+: track 13.5 -> 6.80 mm
- net /d-: track 12.6 -> 6.75 mm
- net Net-(U1-USB_DP): track 2.96 -> 0.00 mm
- net Net-(U1-USB_DM): track 2.62 -> 0.00 mm
