File: person-keyboard.kicad_pcb (KiCad board)
At the start: 2 copper layers, 446.9 x 141.7 mm, 350 parts, among them J1 USB_C_Receptacle_USB2.0_16P, SW1 esc, SW10 f9, SW100 R ctrl, SW101 Left, SW102 down, SW103 right, SW104 num zero, SW105 num full stop, SW107 SW_Push, SW11 f10, SW12 f11, SW13 f12, SW14 prtscr, SW15 scrlck, SW16 pause, SW17 tilde, SW18 1, SW19 2, SW2 f1, SW20 3, SW21 4, SW22 5, SW23 6, SW24 7, SW25 8, SW26 9, SW27 0, SW28 minus, SW29 equals, SW3 f2, SW30 backspace, SW31 insert, SW32 home, SW33 pgup, SW34 num lock, SW35 num slash, SW36 num mult, SW37 num minus, SW38 tab, SW39 q, SW4 f3, SW40 w, SW41 e, SW42 r, SW43 t, SW44 y, SW45 u, SW46 i, SW47 o, SW48 p, SW49 L brac, SW5 f4, SW50 R brac, SW51 enter, SW52 delete, SW53 end, SW54 pgdn, SW55 num 7, SW56 num 8, SW57 num 9, SW58 num add, SW59 capslock, SW6 f5, SW60 a, SW61 s, SW62 d, SW63 f, SW64 g, SW65 h, SW66 j, SW67 k, SW68 l, SW69 sem colon, SW7 f6, SW70 quote, SW71 tilde, SW72 num 4, SW73 num 5, SW74 num 6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

Commit message: Routed microcontroller
Parts:
- added C3: 4.7n, Capacitor_SMD:C_0805_2012Metric_Pad1.18x1.45mm_HandSolder, B.Cu at (415.5, 27.2)
- added SW106: SW_Push, jacob-libs:SW-SMD_L4.0-W2.9-LS5.0, F.Cu at (383.5, 23.0)
- D106: value B340A -> 1N5819; footprint PCM_Diode_SMD_AKL:D_SMA -> Diode_SMD:D_SOD-123
- SW1, SW10, SW100, SW101, SW102, SW103, SW104, SW105, SW11, SW12, SW13, SW14, SW15, SW16, SW17, SW18, SW19, SW2, SW20, SW21, SW22, SW23, SW24, SW25, SW26, SW27, SW28, SW29, SW3, SW31, SW32, SW33, SW34, SW35, SW36, SW37, SW39, SW4, SW40, SW41, SW42, SW43, SW44, SW45, SW46, SW47, SW48, SW49, SW5, SW50, SW52, SW53, SW54, SW55, SW56, SW57, SW6, SW60, SW61, SW62, SW63, SW64, SW65, SW66, SW67, SW68, SW69, SW7, SW70, SW71, SW72, SW73, SW74, SW76, SW77, SW78, SW79, SW8, SW80, SW81, SW82, SW83, SW84, SW85, SW86, SW88, SW89, SW9, SW90, SW91, SW93, SW94, SW95, SW97, SW98, SW99: footprint PCM_Switch_Keyboard_Hotswap_Kailh:SW_Hotswap_Kailh_Choc_V1V2_1.00u -> Gateron_KS33_Hotswap:Gateron-KS33-Hotswap-1U; moved to B.Cu
- SW30: footprint PCM_Switch_Keyboard_Hotswap_Kailh:SW_Hotswap_Kailh_Choc_V1V2_2.00u -> Gateron_KS33_Hotswap:Gateron-KS33-Hotswap-2U; moved to B.Cu
- SW38: footprint PCM_Switch_Keyboard_Hotswap_Kailh:SW_Hotswap_Kailh_Choc_V1V2_1.50u -> Gateron_KS33_Hotswap:Gateron-KS33-Hotswap-1.5U; moved to B.Cu
- SW51, SW58, SW92: footprint PCM_Switch_Keyboard_Hotswap_Kailh:SW_Hotswap_Kailh_Choc_V1V2_2.00u_90deg -> Gateron_KS33_Hotswap:Gateron-KS33-Hotswap-2U-90-Deg; moved to B.Cu
- SW59: footprint PCM_Switch_Keyboard_Hotswap_Kailh:SW_Hotswap_Kailh_Choc_V1V2_1.75u -> Gateron_KS33_Hotswap:Gateron-KS33-Hotswap-1.75U; moved to B.Cu
- SW75: footprint PCM_Switch_Keyboard_Hotswap_Kailh:SW_Hotswap_Kailh_Choc_V1V2_1.25u -> Gateron_KS33_Hotswap:Gateron-KS33-Hotswap-1.25U; moved to B.Cu
- SW87: footprint PCM_Switch_Keyboard_Hotswap_Kailh:SW_Hotswap_Kailh_Choc_V1V2_2.75u -> Gateron_KS33_Hotswap:Gateron-KS33-Hotswap-2.75U; moved to B.Cu
- SW96: footprint PCM_Switch_Keyboard_Hotswap_Kailh:SW_Hotswap_Kailh_Choc_V1V2_6.25u -> Gateron_KS33_Hotswap:Gateron-KS33-Hotswap-6.25U; moved to B.Cu
- U1: footprint Package_DFN_QFN:QFN-56-1EP_7x7mm_P0.4mm_EP3.2x3.2mm -> jacob-libs:QFN-56-1EP_7x7mm_P0.4mm_EP3.2x3.2mm_vias
- moved C1 62.8 mm to (390.4, 25.9), turned to 90 degrees
- moved R7 59.1 mm to (392.3, 37.5), turned to 90 degrees
- moved C9 50.2 mm to (386.5, 39.8), turned to 90 degrees
- moved F1 49.7 mm to (399.2, 22.9)
- moved C13 47.1 mm to (387.5, 39.8), turned to 90 degrees
- moved C11 45.3 mm to (394.7, 49.9), turned to -90 degrees
- moved C10 42.0 mm to (399.0, 48.6), turned to -90 degrees
- moved C14 39.3 mm to (403.5, 44.2), turned to 0 degrees
- moved C8 36.8 mm to (394.7, 37.4), turned to 90 degrees
- moved R1 35.4 mm to (412.2, 32.8), turned to -90 degrees
- moved R2 34.3 mm to (414.1, 32.8), turned to -90 degrees
- moved R6 33.9 mm to (418.6, 27.3), turned to 90 degrees
- moved C6 31.8 mm to (403.5, 43.2), turned to 0 degrees
- moved C4 31.8 mm to (403.5, 39.1), turned to 0 degrees
- moved C12 31.3 mm to (403.5, 37.1), turned to 0 degrees
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Connections:
- C13 pad 2: +1V1 -> GND
- C14 pad 2: +1V1 -> GND
- F1 pad 1: Net-(F1-Pad1) -> VCC
- J1 pad A4: Net-(F1-Pad1) -> VCC
- J1 pad A9: Net-(F1-Pad1) -> VCC
- J1 pad B4: Net-(F1-Pad1) -> VCC
- J1 pad B9: Net-(F1-Pad1) -> VCC
- SW15 pad 1: unconnected-(SW15-Pad1) -> col8
- SW32 pad 1: unconnected-(SW32-Pad1) -> col8
- SW53 pad 1: unconnected-(SW53-Pad1) -> col8
- U4 pad 4: +5V -> VCC
- Y1 pad 3: GND -> Net-(C15-Pad2)
- Y1 pad 4: Net-(C15-Pad2) -> GND
Routing:
- net +3V3: track 0.00 -> 70.2 mm, vias 0 -> 2
- net GND: track 0.00 -> 34.3 mm, vias 0 -> 4
- net Net-(J1-SHIELD): track 0.00 -> 26.3 mm
- net /cs: track 0.00 -> 26.2 mm
- net +1V1: track 0.00 -> 26.1 mm, vias 0 -> 2
- net /sd1: track 0.00 -> 24.1 mm
- net /sd2: track 0.00 -> 22.0 mm
- net VCC: track 0.00 -> 19.0 mm
- net /d-: track 6.75 -> 20.7 mm
- net /d+: track 6.80 -> 20.7 mm
- net Net-(U1-XIN): track 0.00 -> 13.0 mm
- net Net-(J1-CC2): track 0.00 -> 10.4 mm, vias 0 -> 2
- net /sd0: track 0.00 -> 10.2 mm
- net /sd3: track 0.00 -> 10.2 mm
- net /spi_clk: track 0.00 -> 9.80 mm
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- added copper zone on B.Cu, net +3V3
- added copper zone on F.Cu, net GND
Other:
- outline, holes or cut-outs redrawn

Commit message: Started keyboard matrix, completed all rows, completed numpad columns
Parts:
- added D107: 1N4148W, Diode_SMD:D_SOD-123, B.Cu at (452.1, 48.3)
- added J2: i2c display, jacob-libs:0.91 OLED I2C DISPLAY, F.Cu at (431.8, 34.4)
- added R10: 4k8, Resistor_SMD:R_0805_2012Metric_Pad1.20x1.40mm_HandSolder, B.Cu at (426.8, 48.2)
- added R11: 4k8, Resistor_SMD:R_0805_2012Metric_Pad1.20x1.40mm_HandSolder, B.Cu at (428.8, 48.2)
- added REF**: 2U Stabilizer, Keebio-Parts:Gateron-KS33-2u-Stabilizer-Cutout, F.Cu at (295.3, 66.7)
- added REF**: 2U Stabilizer, Keebio-Parts:Gateron-KS33-2u-Stabilizer-Cutout, F.Cu at (288.1, 123.8)
- added REF**: 6.25U, Keebio-Parts:Gateron-KS33-6.25U-Stabilizer-Cutout, F.Cu at (159.5, 142.9)
- added REF**: 2U Stabilizer, Keebio-Parts:Gateron-KS33-2u-Stabilizer-Cutout, F.Cu at (447.7, 133.3)
- added REF**: 2U Stabilizer, Keebio-Parts:Gateron-KS33-2u-Stabilizer-Cutout, F.Cu at (302.4, 95.2)
- added REF**: 2U Stabilizer, Keebio-Parts:Gateron-KS33-2u-Stabilizer-Cutout, F.Cu at (447.7, 95.2)
- added REF**: 2U Stabilizer, Keebio-Parts:Gateron-KS33-2u-Stabilizer-Cutout, F.Cu at (400.1, 142.9)
- added SW108: RotaryEncoder_Switch, Rotary_Encoder:RotaryEncoder_Alps_EC11E-Switch_Vertical_H20mm, F.Cu at (440.4, 35.6)
- SW100, SW93, SW94, SW95, SW97, SW98, SW99: footprint Gateron_KS33_Hotswap:Gateron-KS33-Hotswap-1U -> Gateron_KS33_Hotswap:Gateron-KS33-Hotswap-1.25U
- SW104: footprint Gateron_KS33_Hotswap:Gateron-KS33-Hotswap-1U -> Gateron_KS33_Hotswap:Gateron-KS33-Hotswap-2U
- SW106, SW107: moved to B.Cu
- moved SW106 14.2 mm to (382.3, 37.1), turned to 0 degrees
- moved SW107 13.4 mm to (413.0, 37.6), turned to 0 degrees
- moved D96 12.5 mm to (167.6, 154.9), turned to 0 degrees
- moved D87 12.2 mm to (288.9, 135.3), turned to 0 degrees
- moved D104 12.1 mm to (404.1, 154.9), turned to 0 degrees
- moved D30 12.0 mm to (296.5, 78.1), turned to 0 degrees
- moved R1 10.7 mm to (421.4, 27.2)
- moved D91 10.5 mm to (435.0, 134.2), turned to 90 degrees
- moved D89 9.94 mm to (399.4, 133.0), turned to 90 degrees
- moved D100 9.83 mm to (311.0, 152.0), turned to 90 degrees
- moved D103 9.83 mm to (375.3, 152.0), turned to 90 degrees
- moved D47 9.83 mm to (227.7, 94.9), turned to 90 degrees
- moved D54 9.83 mm to (375.3, 94.9), turned to 90 degrees
- moved D56 9.83 mm to (418.2, 94.9), turned to 90 degrees
- moved D98 9.83 mm to (263.4, 152.0), turned to 90 degrees
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Connections:
- SW105 pad 1: col9 -> col10
- SW36 pad 1: col9 -> col10
- SW37 pad 1: col9 -> col10
- SW57 pad 1: col9 -> col10
- SW58 pad 1: col9 -> col10
- SW74 pad 1: col9 -> col10
- SW91 pad 1: col9 -> col10
- SW92 pad 1: col9 -> col10
- U1 pad 11: unconnected-(U1-GPIO8-Pad11) -> row9
- U1 pad 12: unconnected-(U1-GPIO9-Pad12) -> row8
- U1 pad 13: unconnected-(U1-GPIO10-Pad13) -> row7
- U1 pad 14: unconnected-(U1-GPIO11-Pad14) -> row6
- U1 pad 15: unconnected-(U1-GPIO12-Pad15) -> row5
- U1 pad 16: unconnected-(U1-GPIO13-Pad16) -> row4
- U1 pad 17: unconnected-(U1-GPIO14-Pad17) -> row3
- U1 pad 18: unconnected-(U1-GPIO15-Pad18) -> row2
- U1 pad 2: unconnected-(U1-GPIO0-Pad2) -> sda
- U1 pad 3: unconnected-(U1-GPIO1-Pad3) -> scl
- U1 pad 4: unconnected-(U1-GPIO2-Pad4) -> rot0
- U1 pad 5: unconnected-(U1-GPIO3-Pad5) -> rot1
- U1 pad 6: unconnected-(U1-GPIO4-Pad6) -> col10
- U1 pad 7: unconnected-(U1-GPIO5-Pad7) -> col9
- U1 pad 8: unconnected-(U1-GPIO6-Pad8) -> row11
- U1 pad 9: unconnected-(U1-GPIO7-Pad9) -> row10
Routing:
- net row8: track 0.00 -> 519.6 mm, vias 0 -> 2
- net row10: track 0.00 -> 509.8 mm, vias 0 -> 2
- net row6: track 0.00 -> 464.9 mm, vias 0 -> 2
- net row5: track 0.00 -> 458.3 mm, vias 0 -> 2
- net row9: track 0.00 -> 455.5 mm, vias 0 -> 2
- net row4: track 0.00 -> 454.4 mm, vias 0 -> 2
- net row3: track 0.00 -> 438.7 mm, vias 0 -> 2
- net row2: track 0.00 -> 438.5 mm, vias 0 -> 2
- net row11: track 0.00 -> 426.2 mm
- net row7: track 0.00 -> 421.9 mm, vias 0 -> 2
- net row0: track 0.00 -> 309.6 mm
- net row1: track 0.00 -> 271.5 mm
- net col10: track 0.00 -> 260.0 mm, vias 0 -> 16
- net col9: track 0.00 -> 209.4 mm, vias 0 -> 16
- net rot0: track 0.00 -> 62.0 mm
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- added copper zone on B.Cu, net GND
Other:
- outline, holes or cut-outs redrawn

Commit message: Started Main matrix
Parts:
- moved C1 1.48 mm to (389.4, 27.9)
- moved U2 1.48 mm to (395.9, 27.9)
- moved C8 0.91 mm to (393.9, 36.9), turned to 135 degrees
Connections:
- U1 pad 27: unconnected-(U1-GPIO16-Pad27) -> row1
- U1 pad 28: unconnected-(U1-GPIO17-Pad28) -> row0
- U1 pad 29: unconnected-(U1-GPIO18-Pad29) -> col8
- U1 pad 30: unconnected-(U1-GPIO19-Pad30) -> col7
- U1 pad 31: unconnected-(U1-GPIO20-Pad31) -> col6
- U1 pad 32: unconnected-(U1-GPIO21-Pad32) -> col5
- U1 pad 34: unconnected-(U1-GPIO22-Pad34) -> col4
- U1 pad 35: unconnected-(U1-GPIO23-Pad35) -> col3
- U1 pad 36: unconnected-(U1-GPIO24-Pad36) -> col2
- U1 pad 37: unconnected-(U1-GPIO25-Pad37) -> col1
- U1 pad 38: unconnected-(U1-GPIO26_ADC0-Pad38) -> col0
Routing:
- net col0: track 0.00 -> 593.2 mm, vias 0 -> 6
- net col1: track 0.00 -> 521.9 mm, vias 0 -> 12
- net col2: track 0.00 -> 482.4 mm, vias 0 -> 12
- net col3: track 0.00 -> 447.5 mm, vias 0 -> 12
- net col4: track 0.00 -> 407.9 mm, vias 0 -> 12
- net col5: track 0.00 -> 359.7 mm, vias 0 -> 12
- net col7: track 0.00 -> 298.3 mm, vias 0 -> 10
- net col8: track 0.00 -> 295.3 mm, vias 0 -> 14
- net col6: track 0.00 -> 245.3 mm, vias 0 -> 6
- net row1: track 271.5 -> 380.0 mm, vias 0 -> 2
- net row0: track 309.6 -> 357.5 mm
- net row9: track 455.5 -> 471.3 mm
- net +1V1: track 21.5 -> 25.4 mm, vias 0 -> 2
- net Net-(D90-A): track 0.00 -> 2.72 mm
- net +5V: track 8.05 -> 6.60 mm
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