File: led-backlight.kicad_sch (KiCad schematic)
At the start: 106 parts, among them U5 74AHCT1G125

Commit message: Completed Keyboard matrix, started LED chain
Connections:
- net at SK37.1 (DOUT): now also SK36.3 (DIN)
- net at SK37.3 (DIN): now also SK16.1 (DOUT); no longer SK58.1 (DOUT)
- net at SK35.1 (DOUT): now also SK34.3 (DIN)
- net at SK35.3 (DIN): now also SK36.1 (DOUT); no longer SK56.1 (DOUT)
- net at SK73.1 (DOUT): now also SK72.3 (DIN); no longer SK56.3 (DIN)
- net at SK73.3 (DIN): now also SK74.1 (DOUT); no longer SK90.1 (DOUT)
- net at SK67.1 (DOUT): now also SK66.3 (DIN); no longer SK83.3 (DIN)
- net at SK67.3 (DIN): now also SK68.1 (DOUT); no longer SK46.1 (DOUT)
- net at SK24.1 (DOUT): now also SK23.3 (DIN); no longer SK7.3 (DIN)
- net at SK24.3 (DIN): now also SK25.1 (DOUT); no longer SK45.1 (DOUT)
- net at SK11.1 (DOUT): now also SK12.3 (DIN); no longer SK29.3 (DIN)
- net at SK100.1 (DOUT): now also SK99.3 (DIN); no longer SK87.3 (DIN)
- net at SK100.3 (DIN): now also SK101.1 (DOUT); no longer SK99.1 (DOUT)
- net at SK103.1 (DOUT): now also SK102.3 (DIN); no longer SK54.3 (DIN)
- net at SK103.3 (DIN): now also SK104.1 (DOUT); no longer SK102.1 (DOUT)
- net at SK15.1 (DOUT): now also SK16.3 (DIN); no longer SK32.3 (DIN)
- net at SK22.1 (DOUT): now also SK21.3 (DIN); no longer SK5.3 (DIN)
- net at SK22.3 (DIN): now also SK23.1 (DOUT); no longer SK43.1 (DOUT)
- net at SK72.1 (DOUT): now also SK71.3 (DIN); no longer SK89.3 (DIN)
- net at SK55.1 (DOUT): now also SK56.3 (DIN); no longer SK72.3 (DIN)
- net at SK52.1 (DOUT): now also SK53.3 (DIN); no longer SK31.3 (DIN)
- net at SK52.3 (DIN): now also SK51.1 (DOUT); no longer SK101.1 (DOUT)
- net at SK88.1 (DOUT): now also SK89.3 (DIN); no longer SK102.3 (DIN)
- net at SK46.3 (DIN): now also SK45.1 (DOUT); no longer SK25.1 (DOUT)
- net at SK82.1 (DOUT): now also SK83.3 (DIN); no longer SK66.3 (DIN)
- net at SK82.3 (DIN): now also SK81.1 (DOUT); no longer SK96.1 (DOUT)
- net at SK1.1 (DOUT): now also SK2.3 (DIN); no longer SK17.3 (DIN)
- net at SK71.1 (DOUT): now also SK70.3 (DIN); no longer SK99.3 (DIN)
- net at SK58.3 (DIN): now also SK57.1 (DOUT); no longer SK92.1 (DOUT)
- net at SK96.3 (DIN): now also SK97.1 (DOUT); no longer SK81.1 (DOUT)
- net at SK98.1 (DOUT): now also SK97.3 (DIN); no longer SK86.3 (DIN)
- net at SK98.3 (DIN): now also SK99.1 (DOUT); no longer SK97.1 (DOUT)
- net at SK18.1 (DOUT): now also SK17.3 (DIN); no longer SK2.3 (DIN)
- net at SK18.3 (DIN): now also SK19.1 (DOUT); no longer SK39.1 (DOUT)
- net at SK87.1 (DOUT): now also SK88.3 (DIN); no longer SK12.3 (DIN)
- net at SK4.1 (DOUT): now also SK5.3 (DIN); no longer SK21.3 (DIN)
- net at SK44.3 (DIN): now also SK43.1 (DOUT); no longer SK23.1 (DOUT)
- net at SK6.1 (DOUT): now also SK7.3 (DIN); no longer SK23.3 (DIN)
- net at SK53.1 (DOUT): now also SK54.3 (DIN); no longer SK88.3 (DIN)
- net at SK32.1 (DOUT): now also SK31.3 (DIN); no longer SK53.3 (DIN)
- net at SK47.1 (DOUT): now also SK48.3 (DIN); no longer SK26.3 (DIN)
- net at SK47.3 (DIN): now also SK46.1 (DOUT); no longer SK68.1 (DOUT)
- net at SK39.3 (DIN): now also SK38.1 (DOUT); no longer SK60.1 (DOUT)
- net at SK91.3 (DIN): now also SK90.1 (DOUT); no longer SK74.1 (DOUT)
- net at SK74.3 (DIN): now also SK58.1 (DOUT); no longer SK57.1 (DOUT)
- net at SK26.1 (DOUT): now also SK25.3 (DIN); no longer SK9.3 (DIN)
- net at SK41.1 (DOUT): now also SK42.3 (DIN); no longer SK20.3 (DIN)
- net at SK41.3 (DIN): now also SK40.1 (DOUT); no longer SK62.1 (DOUT)
- net at SK60.3 (DIN): now also SK61.1 (DOUT); no longer SK76.1 (DOUT)
- net at SK68.3 (DIN): now also SK69.1 (DOUT); no longer SK84.1 (DOUT)
- net at SK57.3 (DIN): now also SK56.1 (DOUT); no longer SK36.1 (DOUT)
- net at SK33.1 (DOUT): now also SK32.3 (DIN); no longer SK16.3 (DIN)
- net at SK76.3 (DIN): now also SK75.1 (DOUT); no longer SK94.1 (DOUT)
- net at SK45.3 (DIN): now also SK44.1 (DOUT); no longer SK66.1 (DOUT)
- net at SK79.3 (DIN): now also SK78.1 (DOUT); no longer SK63.1 (DOUT)
- net at SK70.1 (DOUT): now also SK69.3 (DIN); no longer SK49.3 (DIN)
- net at SK86.1 (DOUT): now also SK87.3 (DIN); no longer SK70.3 (DIN)
- net at SK50.1 (DOUT): now also SK51.3 (DIN); no longer SK71.3 (DIN)
- net at SK50.3 (DIN): now also SK49.1 (DOUT); no longer SK29.1 (DOUT)
- net at SK30.1 (DOUT): now also SK29.3 (DIN); no longer SK51.3 (DIN)
- net at SK30.3 (DIN): now also SK31.1 (DOUT); no longer SK13.1 (DOUT)
- net at SK8.1 (DOUT): now also SK9.3 (DIN); no longer SK25.3 (DIN)
- net at SK54.1 (DOUT): now also SK55.3 (DIN); no longer SK33.3 (DIN)
- net at SK3.3 (DIN): now also SK2.1 (DOUT); no longer SK20.1 (DOUT)
- net at SK40.3 (DIN): now also SK39.1 (DOUT); no longer SK19.1 (DOUT)
- net at SK19.3 (DIN): now also SK20.1 (DOUT); no longer SK2.1 (DOUT)
- net at SK85.3 (DIN): now also SK84.1 (DOUT); no longer SK69.1 (DOUT)
- net at SK48.1 (DOUT): now also SK49.3 (DIN); no longer SK69.3 (DIN)
- net at SK90.3 (DIN): now also SK89.1 (DOUT); no longer SK104.1 (DOUT)
- net at SK104.3 (DIN): now also SK105.1 (DOUT); no longer SK89.1 (DOUT)
- net at SK43.3 (DIN): now also SK42.1 (DOUT); no longer SK64.1 (DOUT)
- net at SK28.3 (DIN): now also SK29.1 (DOUT); no longer SK49.1 (DOUT)
- net at SK95.1 (DOUT): now also SK94.3 (DIN); no longer SK78.3 (DIN)
- net at SK95.3 (DIN): now also SK96.1 (DOUT); no longer SK77.1 (DOUT)
- net at SK9.1 (DOUT): now also SK10.3 (DIN); no longer SK27.3 (DIN)
- net at SK91.1 (DOUT): now also SK92.3 (DIN); no longer SK105.3 (DIN)
- net at SK80.1 (DOUT): now also SK81.3 (DIN); no longer SK64.3 (DIN)
- net at SK62.3 (DIN): now also SK63.1 (DOUT); no longer SK78.1 (DOUT)
- net at SK85.1 (DOUT): now also SK86.3 (DIN); no longer SK97.3 (DIN)
- net at SK65.3 (DIN): now also SK66.1 (DOUT); no longer SK44.1 (DOUT)
- net at SK65.1 (DOUT): now also SK64.3 (DIN); no longer SK81.3 (DIN)
- net at SK27.1 (DOUT): now also SK26.3 (DIN); no longer SK48.3 (DIN)
- net at SK77.3 (DIN): now also SK76.1 (DOUT); no longer SK61.1 (DOUT)
- net at SK61.3 (DIN): now also SK62.1 (DOUT); no longer SK40.1 (DOUT)
- net at SK34.1 (DOUT): now also SK33.3 (DIN); no longer SK55.3 (DIN)
- net at SK14.3 (DIN): now also SK13.1 (DOUT); no longer SK31.1 (DOUT)
- net at SK93.1 (DOUT): no longer SK94.3 (DIN)
- net at SK63.3 (DIN): now also SK64.1 (DOUT); no longer SK42.1 (DOUT)
- net at SK101.3 (DIN): now also SK102.1 (DOUT); no longer SK51.1 (DOUT)
- net at SK21.1 (DOUT): now also SK20.3 (DIN); no longer SK42.3 (DIN)
- net at SK28.1 (DOUT): now also SK27.3 (DIN); no longer SK10.3 (DIN)
- net at SK59.3 (DIN): now also SK60.1 (DOUT); no longer SK38.1 (DOUT)
- net at SK93.3 (DIN): now also SK94.1 (DOUT); no longer SK75.1 (DOUT)
- new net: SK77.1 (DOUT), SK78.3 (DIN)
- new net: SK105.3 (DIN), SK92.1 (DOUT)
- no-connect marks 1 -> 0
